File: YTAR/YTAR.kicad_sch (KiCad schematic)
At the start: 37 parts, among them J1 STDC14, SW1 Tact, U1 STM32H750XBHx, Y1 25MHz

Commit message: DRAM added
Parts:
- removed U1: STM32H750XBHx, Package_BGA:TFBGA-265_14x14mm_Layout17x17_P0.8mm, symbol MCU_ST_STM32H7:STM32H750XBHx
- added C29, C30, C31, C32, C33, C34, C35, C36, C37, C38, C39, C40, C41, C42, C43: 100n, Capacitor_SMD:C_0402_1005Metric, symbol MEMS_CAPACITORS:C_100n_0402_16V_X7R_MLASE105SB7104KFNA01
- added J2: Conn_2x04_2.54mm_male_vertical, Connector_PinSocket_2.54mm:PinSocket_2x04_P2.54mm_Vertical, symbol MEMS_ELECTROMECHANICAL:Conn_2x04_2.54mm_male_vertical
- added JP1, JP2, JP3, JP4: ~, MEMS_Passive:R_0805_2012Metric_Jumper_Open, symbol MEMS_PASSIVE:SolderableJumper_Open
- added JP5: CAN, MEMS_Passive:R_0805_2012Metric_Jumper_Open, symbol MEMS_PASSIVE:SolderableJumper_Open
- added R1, R10, R11, R12, R13, R14, R15, R16, R17, R18, R19, R2, R3, R4, R5, R6, R7, R8, R9: 10k, Resistor_SMD:R_0402_1005Metric, symbol MEMS_RESISTORS_0402:R_10k_0402_1%_50ppm_RT0402FRE0710KL
- added R20: 120R, Resistor_SMD:R_0402_1005Metric, symbol MEMS_RESISTORS_0402:R_120R_0402_1%_50ppm_RT0402FRE07120RL
- added R21: 620R, Resistor_SMD:R_0402_1005Metric, symbol MEMS_RESISTORS_0402:R_620R_0402_1%_50ppm_RT0402FRE07620RL
- added R22: 100R, Resistor_SMD:R_0402_1005Metric, symbol MEMS_RESISTORS_0402:R_100R_0402_1%_50ppm_RT0402FRE07100RL
- added U1: STM32H750XBHx, Package_BGA:TFBGA-265_14x14mm_Layout17x17_P0.8mm, symbol MEMS_IC:STM32H750XBHx
- added U2: MCP2562-E-MF, Package_DFN_QFN:DFN-8-1EP_3x3mm_P0.65mm_EP1.55x2.4mm, symbol Interface_CAN_LIN:MCP2562-E-MF
- added U3: DS90C124, Package_QFP:TQFP-48_7x7mm_P0.5mm, symbol MEMS_IC:DS90C124
- added U4: ~, Package_BGA:BGA-90_8.0x13.0mm_Layout2x3x15_P0.8mm, symbol MEMS_IC:IS42S32400F-6BL
- TP2: value MCU_3V3 -> 3V3
Connections:
- net +3.3V: now also JP1.1, JP2.1, JP3.1, JP4.1; no longer C26.1, C27.1
- net FD_CAN1_RX: now also U1.B17 (PH14)
- net FD_CAN1_TX: now also U1.D4 (PB9)
- net GND: now also C29.2, C30.2, C31.2, C32.2, C33.2, C34.2, C35.2, C36.2, C37.2, C38.2, C39.2, C40.2, C41.2, C42.2, C43.2, R1.2, R10.2, R11.2, R12.2, R13.2, R14.2, R15.2, R16.2, R17.1, R18.1, R19.1, R2.2, R3.2, R4.2, R5.2, R6.2, R7.2, R8.2, R9.2, U1.A1 (VSS), U1.A17 (VSS), U1.B2 (VSS), U1.B6 (VSS), U1.C10 (VSS), U1.C13 (VSS), U1.C16 (VSS), U1.F1 (VSS), U1.F2 (VSS), U1.G10 (VSS), U1.G11 (VSS), U1.G16 (VSS), U1.G2 (VSS), U1.G7 (VSS), U1.G8 (VSS), U1.G9 (VSS), U1.H10 (VSS), U1.H11 (VSS), U1.H7 (VSS), U1.H8 (VSS), U1.H9 (VSS), U1.J10 (VSS), U1.J11 (VSS), U1.J16 (VSS), U1.J17 (VSS), U1.J3 (VSS), U1.J7 (VSS), U1.J8 (VSS), U1.J9 (VSS), U1.K10 (VSS), U1.K11 (VSS), U1.K15 (VSS), U1.K7 (VSS), U1.K8 (VSS), U1.K9 (VSS), U1.L10 (VSS), U1.L11 (VSS), U1.L15 (VSS), U1.L7 (VSS), U1.L8 (VSS), U1.L9 (VSS), U1.M15 (VSS), U1.N16 (VSS), U1.P1 (VSSA), U1.R4 (VSS), U1.R8 (VSS), U1.T12 (VSS), U1.U1 (VSS), U1.U17 (VSS), U2.2 (VSS), U2.9 (PAD), U4.A3 (VSS), U4.B3 (VSSQ), U4.B8 (VSSQ), U4.C1 (VSSQ), U4.D1 (VSSQ), U4.E9 (VSSQ), U4.F1 (VSS), U4.L3 (VSS), U4.L9 (VSSQ), U4.M1 (VSSQ), U4.N1 (VSSQ), U4.P3 (VSSQ), U4.P8 (VSSQ), U4.R3 (VSS)
- net JCLK/SWCLK: now also U1.B14 (PA14)
- net JTDI/SWO: now also U1.A14 (PA15)
- net JTDO/SWO: now also U1.C6 (PB3)
- net JTMS/SWDIO: now also U1.C15 (PA13)
- net RCC_IN: now also U1.J2 (PH0)
- net RCC_OUT: now also U1.J1 (PH1)
- net VDD_33_USB: now also U1.F17 (VDD33_USB)
- net VDD_50_USB: now also U1.G17 (VDD50_USB)
- net ~{STM_RST}: now also U1.K1 (NRST)
- net at C25.1: now also U1.A6 (VDDLDO), U1.C17 (VDDLDO), U1.U12 (VDDLDO)
- net at C1.1, C2.1: now also U1.A7 (VCAP), U1.D17 (VCAP), U1.U11 (VCAP)
- new net: R18.2, U4.F8 (DQM2)
- new net: R3.1, U4.D2 (DQ29)
- new net: R7.1, U4.C3 (DQ25)
- new net: R6.1, U4.A1 (DQ26)
- new net: R8.1, U4.A2 (DQ24)
- new net: R9.1, U4.A8 (DQ23)
- new net: R11.1, U4.A9 (DQ21)
- new net: R4.1, U4.B1 (DQ28)
- new net: R13.1, U4.B9 (DQ19)
- new net: R5.1, U4.C2 (DQ27)
- new net: R10.1, U4.C7 (DQ22)
- new net: R12.1, U4.C8 (DQ20)
- new net: R2.1, U4.D3 (DQ30)
- new net: R15.1, U4.D7 (DQ17)
- new net: R14.1, U4.D8 (DQ18)
- new net: R1.1, U4.E2 (DQ31)
- new net: R16.1, U4.E8 (DQ16)
- new net: R17.2, U4.F2 (DQM3)
- new net: JP5.2, R20.2
- new net: R19.2, U2.8 (SHDN)
- new net A0: U4.G8 (A0)
- new net A1: U4.G9 (A1)
- new net A10: U4.G7 (A10)
- new net A11: U4.H9 (A11)
- new net A2: U4.F7 (A2)
- new net A3: U4.F3 (A3)
- new net A4: U4.G1 (A4)
- new net A5: U4.G2 (A5)
- new net A6: U4.G3 (A6)
- new net A7: U4.H1 (A7)
- new net A8: U4.H2 (A8)
- new net A9: U4.J3 (A9)
- new net BA0: U4.J7 (BA0)
- new net BA1: U4.H8 (BA1)
- new net CAM_CAN_H: J2.8 (Pin_8)
- new net CAM_CAN_L: J2.7 (Pin_7)
- new net CAM_GND: J2.6 (Pin_6)
- new net CAM_LVDS_H: J2.2 (Pin_2)
- new net CAM_LVDS_L: J2.1 (Pin_1)
- new net CAM_VCC: J2.5 (Pin_5)
- new net CAN_H: R20.1, U2.7 (CANH)
- new net CAN_L: JP5.1, U2.6 (CANL)
- new net CAN_RX: U2.4 (RXD)
- new net CAN_TX: U2.1 (TXD)
- new net DQ0: U4.R8 (DQ0)
- new net DQ1: U4.N7 (DQ1)
- new net DQ10: U4.M2 (DQ10)
- new net DQ11: U4.P1 (DQ11)
- new net DQ12: U4.N2 (DQ12)
- new net DQ13: U4.R1 (DQ13)
- new net DQ14: U4.N3 (DQ14)
- new net DQ15: U4.R2 (DQ15)
- new net DQ2: U4.R9 (DQ2)
- new net DQ3: U4.N8 (DQ3)
- new net DQ4: U4.P9 (DQ4)
- new net DQ5: U4.M8 (DQ5)
- new net DQ6: U4.M7 (DQ6)
- new net DQ7: U4.L8 (DQ7)
- new net DQ8: U4.L2 (DQ8)
- new net DQ9: U4.M3 (DQ9)
- new net NBL0: U4.K9 (DQM0)
- new net NBL1: U4.K1 (DQM1)
- new net SDN_CAS: U4.K7 (~{CAS})
- new net SDN_CKE: U4.J2 (CKE)
- new net SDN_CLK: U4.J1 (CLK)
- new net SDN_NE: U4.J8 (~{CS})
- new net SDN_RAS: U4.J9 (~{RAS})
- new net SDN_WE: U4.K8 (~{WE})
- new net VDD_CAN: C43.1, JP4.2, U2.3 (VDD), U2.5 (Vio)
- new net VDD_DES: JP3.2
- new net VDD_DRAM: C29.1, C30.1, C31.1, C32.1, C33.1, C34.1, C35.1, C36.1, C37.1, C38.1, C39.1, C40.1, C41.1, C42.1, JP2.2, U4.A7 (VDD), U4.B2 (VDDQ), U4.B7 (VDDQ), U4.C9 (VDDQ), U4.D9 (VDDQ), U4.E1 (VDDQ), U4.F9 (VDD), U4.L1 (VDDQ), U4.L7 (VDD), U4.M9 (VDDQ), U4.N9 (VDDQ), U4.P2 (VDDQ), U4.P7 (VDDQ), U4.R7 (VDD)
- new net VDD_MCU: C26.1, C27.1, JP1.2, U1.E11 (VDD), U1.E6 (VDD), U1.E9 (VDD), U1.F5 (VDD), U1.G13 (VDD), U1.G5 (VDD), U1.H13 (VDD), U1.H5 (VDD), U1.J13 (VDD), U1.K13 (VDD), U1.K5 (VDD), U1.L1 (VDDA), U1.L13 (VDD), U1.L5 (VDD), U1.M13 (VDD), U1.M5 (VDD), U1.N10 (VDD), U1.N11 (VDD), U1.N12 (VDD), U1.N7 (VDD), U1.N8 (VDD), U1.P17 (VDD)
- no-connect marks 0 -> 6
Other:
- note added: "Per every VDD pin"
- note added: "ZAMIENIĆ NA COŚ FAJNEGO"
- moved on the sheet: D1, D2, D3

Commit message: Added more things
Parts:
- removed R22: 100R, Resistor_SMD:R_0402_1005Metric, symbol MEMS_RESISTORS_0402:R_100R_0402_1%_50ppm_RT0402FRE07100RL
- added C44, C45, C46, C47, C48, C49, C50, C51, C52, C53: 100n, Capacitor_SMD:C_0402_1005Metric, symbol MEMS_CAPACITORS:C_100n_0402_16V_X7R_MLASE105SB7104KFNA01
- added JP6: DES_CLS_SEL, MEMS_Passive:R_0805_2012Metric_Jumper_Open, symbol MEMS_PASSIVE:SolderableJumper_Open
- added R22, R24: 49R9, Resistor_SMD:R_0402_1005Metric, symbol MEMS_RESISTORS_0402:R_49R9_0402_1%_50ppm_RT0402FRE0749R9L
- added R23: 10k, Resistor_SMD:R_0402_1005Metric, symbol MEMS_RESISTORS_0402:R_10k_0402_1%_50ppm_RT0402FRE0710KL
Connections:
- net +3.3V: no longer J1.3 (VCC)
- net CAM_LVDS_H: now also C44.1
- net CAM_LVDS_L: now also C45.1
- net GND: now also U3.19 (VSSOR2), U3.2 (RESRVD), U3.29 (VSSOR1), U3.35 (VSSR0), U3.38 (VSSR1), U3.40 (VSSIR), U3.44 (VSSPR1), U3.46 (VSSPR0), U3.7 (VDDOR3), C46.2, C47.2, C48.2, C49.2, C50.2, C51.2, C52.2, C53.2, JP6.1
- net VDD_DES: now also U3.1 (RPWDNB), U3.20 (VDDOR2), U3.30 (VDDOR1), U3.36 (VDDR0), U3.37 (VDDR1), U3.39 (VDDIR), U3.45 (VDDPR1), U3.47 (VDDPR0), U3.48 (REN), U3.8 (VSSOR3), C46.1, C47.1, C48.1, C49.1, C50.1, C51.1, C52.1, C53.1, R23.2
- net VDD_MCU: now also J1.3 (VCC)
- net ROUT15: now reaches U3.13 (ROUT15)
- net ROUT14: now reaches U3.14 (ROUT14)
- net ROUT13: now reaches U3.15 (ROUT13)
- net ROUT12: now reaches U3.16 (ROUT12)
- net DES_LOCK: now reaches U3.17 (LOCK)
- net DES_RCLK: now reaches U3.18 (RCLK)
- net ROUT11: now reaches U3.21 (ROUT11)
- net ROUT10: now reaches U3.22 (ROUT10)
- net ROUT9: now reaches U3.23 (ROUT9)
- net ROUT8: now reaches U3.24 (ROUT8)
- net ROUT7: now reaches U3.25 (ROUT7)
- net ROUT6: now reaches U3.26 (ROUT6)
- net ROUT5: now reaches U3.27 (ROUT5)
- net ROUT4: now reaches U3.28 (ROUT4)
- net ROUT3: now reaches U3.31 (ROUT3)
- net ROUT2: now reaches U3.32 (ROUT2)
- net ROUT1: now reaches U3.33 (ROUT1)
- net ROUT0: now reaches U3.34 (ROUT0)
- net at U3.41 (RIN+): now also C44.2, R22.1
- net at U3.42 (RIN-): now also C45.2, R24.2
- net DES_RRFB: now reaches U3.43 (RRFB)
- net DES_RRFB: now also JP6.2, R23.1
- new net: R22.2, R24.1
- no-connect marks 6 -> 14
Other:
- note added: "Dodaj 4.7nF"
- moved on the sheet: C29, C30, C31, C32, C33, C34, C35, C36, C37, C38, C39, C40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

Commit message: SDRAM podłączony. Dodane rezystory na liniach
Parts:
- added R25, R26, R27, R28, R29, R30, R31, R32, R33, R34, R35, R36, R37, R38, R39, R40, R41, R42, R43, R44, R45, R46, R47, R48, R49, R50, R51, R52, R53, R54, R55, R56, R57, R58, R59, R60, R61: 33R, Resistor_SMD:R_0402_1005Metric, symbol MEMS_RESISTORS_0402:R_33R_0402_1%_50ppm_RT0402FRE0733RL
Connections:
- net A0: now also R42.2
- net A1: now also R43.2
- net A10: now also R56.1
- net A11: now also R57.1
- net A2: now also R44.2
- net A3: now also R45.2
- net A4: now also R46.2
- net A5: now also R47.2
- net A6: now also R49.2
- net A7: now also R50.2
- net A8: now also R51.2
- net A9: now also R52.2
- net BA0: now also R58.1
- net BA1: now also R59.1
- net DQ0: now also R25.2
- net DQ1: now also R26.2
- net DQ10: now also R40.2
- net DQ11: now also R41.2
- net DQ12: now also U1.R11 (PE15)
- net DQ13: now also R29.2
- net DQ14: now also R30.2
- net DQ15: now also R31.2
- net DQ2: now also R27.2
- net DQ3: now also R28.2
- net DQ4: now also R34.2
- net DQ5: now also R35.2
- net DQ6: now also R36.2
- net DQ7: now also R37.2
- net DQ8: now also R38.2
- net DQ9: now also R39.2
- net NBL0: now also R32.2
- net NBL1: now also R33.2
- net SDN_CAS: now also R61.1
- net SDN_CKE: now also R55.1
- net SDN_CLK: now also R60.1
- net SDN_NE: now also R54.1
- net SDN_RAS: now also R48.2
- net SDN_WE: now also R53.1
- net at U1.B4 (PE1): now also R33.1
- net at U1.C1 (PC15): now also R26.1
- net at U1.C2 (PC14): now also R25.1
- net at U1.C4 (PE0): now also R32.1
- net at U1.D13 (PD0): now also R27.1
- net at U1.D6 (PG15): now also R61.2
- net at U1.E12 (PD1): now also R28.1
- net at U1.F15 (PG8): now also R60.2
- net at U1.G1 (PF2): now also R44.1
- net at U1.G14 (PG5): now also R59.2
- net at U1.G3 (PF1): now also R43.1
- net at U1.G4 (PF0): now also R42.1
- net at U1.H14 (PG4): now also R58.2
- net at U1.H4 (PF3): now also R45.1
- net at U1.J4 (PF5): now also R47.1
- net at U1.J5 (PF4): now also R46.1
- net at U1.N9 (PE10): now also R37.1
- net at U1.P10 (PE11): now also R38.1
- net at U1.P4 (PH5): now also R53.2
- net at U1.P7 (PF13): now also R50.1
- net at U1.P8 (PF14): now also R51.1
- net at U1.P9 (PE9): now also R36.1
- net at U1.R10 (PE12): now also R39.1
- net at U1.R7 (PF12): now also R49.1
- net at U1.R9 (PF15): now also R52.1
- net at U1.T10 (PE13): now also R40.1
- net at U1.T11 (PH6): now also R54.2
- net at U1.T16 (PD10): now also R31.1
- net at U1.T17 (PD9): now also R30.1
- net at U1.T7 (PF11): now also R48.1
- net at U1.T8 (PG0): now also R56.2
- net at U1.T9 (PE8): now also R35.1
- net at U1.U10 (PE14): now also R41.1
- net at U1.U13 (PH7): now also R55.2
- net at U1.U16 (PD8): now also R29.1
- net at U1.U8 (PG1): now also R57.2
- net at U1.U9 (PE7): now also R34.1
Other:
- moved on the sheet: R1, R10, R11, R12, R13, R14, R15, R16, R17, R18, R2, R3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

Commit message: Podłączono kwarc
Parts:
- added C54: 2.2u, Capacitor_SMD:C_0402_1005Metric, symbol MEMS_CAPACITORS:C_2u2_0402_10V_X5R_LMK105ABJ225KVHF
- added C55: 4.7n, Capacitor_SMD:C_0402_1005Metric, symbol MEMS_CAPACITORS:C_4n7_0402_50V_X7R_04025C472KAT2A
- added C56, C57: 8.2p, Capacitor_SMD:C_0402_1005Metric, symbol MEMS_CAPACITORS:C_8p2_0402_50V_C0G_04025A8R2CAT2A_
- added J5: USB_C_USB4085-GF-A, Connector_USB:USB_C_Receptacle_GCT_USB4085, symbol MEMS_ELECTROMECHANICAL:USB_C_USB4085-GF-A
- added JP7: BOOT, MEMS_Passive:R_0805_2012Metric_Jumper_Open, symbol MEMS_PASSIVE:SolderableJumper_Open
- added R62, R63: 620R, Resistor_SMD:R_0402_1005Metric, symbol MEMS_RESISTORS_0402:R_620R_0402_1%_50ppm_RT0402FRE07620RL
- added R64, R65: 10k, Resistor_SMD:R_0402_1005Metric, symbol MEMS_RESISTORS_0402:R_10k_0402_1%_50ppm_RT0402FRE0710KL
- added R66: 0R, Resistor_SMD:R_0402_1005Metric, symbol MEMS_RESISTORS:R_0R_0402_RMC1/16SJPTH
- added TP3, TP4: 3V3, MEMS_Custom:TestPoint_Pad_D1.0mm, symbol MEMS_ELECTROMECHANICAL:TestPoint
- JP6: value DES_CLS_SEL -> DES_CLK_SEL
Connections:
- net VDD_33_USB is gone; now on net VDDA: U1.F17 (VDD33_USB)
- net VDD_50_USB is gone; now on net VDDA: U1.G17 (VDD50_USB)
- net VDD_MCU is gone; now on net VDDA: C26.1, C27.1, J1.3 (VCC), JP1.2, U1.E11 (VDD), U1.E6 (VDD), U1.E9 (VDD), U1.F5 (VDD), U1.G13 (VDD), U1.G5 (VDD), U1.H13 (VDD), U1.H5 (VDD), U1.J13 (VDD), U1.K13 (VDD), U1.K5 (VDD), U1.L1 (VDDA), U1.L13 (VDD), U1.L5 (VDD), U1.M13 (VDD), U1.M5 (VDD), U1.N10 (VDD), U1.N11 (VDD), U1.N12 (VDD), U1.N7 (VDD), U1.N8 (VDD), U1.P17 (VDD)
- net +3.3V: now also D1.2 (A), D2.2 (A), D3.2 (A)
- net GND: now also R21.2, U1.N1 (VREF-), Y1.2, Y1.4, C54.2, C55.1, C56.2, C57.2, J5.A1 (GND), J5.A12 (GND), J5.B1 (GND), J5.B12 (GND), J5.S1 (SHIELD), R65.1
- net RCC_IN: now also R66.1
- net RCC_OUT: now also Y1.3, C57.1
- net at R22.2, R24.1: now also C55.2
- net at R21.1: now also D3.1 (K)
- net at Y1.1: now also C56.1, R66.2
- net VDDA: now reaches C25.1, U1.A6 (VDDLDO), U1.C17 (VDDLDO), U1.U12 (VDDLDO)
- net VDDA: now also U1.B1 (VBAT), U1.M1 (VREF+), C54.1, JP7.2, R64.2
- net at U1.E7 (PDR_ON): now also R64.1
- net BOOT0: now reaches U1.E8 (BOOT0)
- net BOOT0: now also JP7.1, R65.2
- net at D2.1 (K): now also R63.1
- net at D1.1 (K): now also R62.1
- new net: J5.A4 (VBUS), J5.A9 (VBUS), J5.B4 (VBUS), J5.B9 (VBUS)
- new net D+: J5.A6 (D+), J5.B6 (D+), TP4.1
- new net D-: J5.A7 (D-), J5.B7 (D-), TP3.1
Other:
- note added: "DODAĆ DO BIBLIOTEKI"
- note added: "Dokończ!"
- note added: "POWER"
- note added: "Pododawać testpointy"
- note added: "VBAT tymczasowo do 3V3"
- note removed: "Dodaj 4.7nF"
- moved on the sheet: C26, C27, JP6, R23, Y1

Commit message: Basic layout
Parts:
- removed J2: Conn_2x04_2.54mm_male_vertical, Connector_PinSocket_2.54mm:PinSocket_2x04_P2.54mm_Vertical, symbol MEMS_ELECTROMECHANICAL:Conn_2x04_2.54mm_male_vertical
- removed SW1: Tact, Button_Switch_SMD:SW_SPST_B3S-1000, symbol MEMS_ELECTROMECHANICAL:SW_Push_Tact_B3S-1000
- removed TP3, TP4: 3V3, MEMS_Custom:TestPoint_Pad_D1.0mm, symbol MEMS_ELECTROMECHANICAL:TestPoint
- added J2: CAMERA, Connector_Hirose:Hirose_DF52-8S-0.8H_1x08-1MP_P0.80mm_Horizontal, symbol MEMS_ELECTROMECHANICAL:DF52-8S-0.8H
- added J3: Micro_Sd, Connector_Card:microSD_HC_Hirose_DM3AT-SF-PEJM5, symbol MEMS_ELECTROMECHANICAL:SD_HC_Hirose_DM3AT-SF-PEJM5
- added J6: IO, Connector_Hirose:Hirose_DF52-8S-0.8H_1x08-1MP_P0.80mm_Horizontal, symbol MEMS_ELECTROMECHANICAL:DF52-8S-0.8H
- added R67, R68: 5k1, Resistor_SMD:R_0402_1005Metric, symbol MEMS_RESISTORS_0402:R_5k1_0402_1%_50ppm_RT0402FRE075K1L
- added SW1: Tact, Button_Switch_SMD:SW_SPST_B3U-1000P, symbol MEMS_ELECTROMECHANICAL:SW_Push_Tact_B3U-1000PM
- added U5: TPS56339, Package_TO_SOT_SMD:TSOT-23-6, symbol MEMS_IC:TPS56339
Connections:
- net +3.3V: no longer C10.1, C11.1, C12.1, C13.1, C14.1, C15.1, C16.1, C17.1, C18.1, C19.1, C20.1, C21.1, C22.1, C23.1, C24.1, C3.1, C4.1, C5.1, C6.1, C7.1, C8.1, C9.1
- net CAM_CAN_H: now also J2.5 (Pin_5)
- net CAM_CAN_L: now also J2.6 (Pin_6)
- net CAM_LVDS_H: now also J2.3 (Pin_3)
- net CAM_LVDS_L: now also J2.4 (Pin_4)
- net D+: now also U1.E16 (PA12)
- net D-: now also U1.E17 (PA11)
- net GND: now also J2.2 (Pin_2), J6.2 (Pin_2), R67.2, R68.2, SW1.1
- net VDDA: now also C10.1, C11.1, C12.1, C13.1, C14.1, C15.1, C16.1, C17.1, C18.1, C19.1, C20.1, C21.1, C22.1, C23.1, C24.1, C3.1, C4.1, C5.1, C6.1, C7.1, C8.1, C9.1
- net ~{STM_RST}: now also SW1.2
- net at J5.A5 (CC1): now also R67.1
- net at J5.B5 (CC2): now also R68.1
- new net +12V_CAM: J2.1 (Pin_1)
- new net +12V_IN: J6.1 (Pin_1)
- no-connect marks 14 -> 17
Other:
- note added: "Sprawdz piny USB"
- moved on the sheet: J5

Commit message: Added LCD labels and corredted SRAM
Parts:
- added J4: FH12-40S-0.5SH(55), Connector_FFC-FPC:Hirose_FH12-40S-0.5SH_1x40-1MP_P0.50mm_Horizontal, symbol MEMS_ELECTROMECHANICAL:FH12-40S-0.5SH(55)
- added SW2: PICTURE, Button_Switch_SMD:SW_SPST_B3U-1000P, symbol MEMS_ELECTROMECHANICAL:SW_Push_Tact_B3U-1000PM
- added SW3: MODE, Button_Switch_SMD:SW_SPST_B3U-1000P, symbol MEMS_ELECTROMECHANICAL:SW_Push_Tact_B3U-1000PM
- added TP10, TP11, TP3, TP4, TP5, TP6, TP7, TP8, TP9: ~, MEMS_Custom:TestPoint_Pad_D1.0mm, symbol MEMS_ELECTROMECHANICAL:TestPoint
- SW1: value Tact -> RESET
Connections:
- net +5V: now also J4.25 (Pin_25), J4.26 (Pin_26)
- net DES_LOCK: now also U1.N4 (PA1)
- net DES_RCLK: now also U1.N5 (PA0)
- net GND: now also J4.27 (Pin_27), J4.40 (Pin_40)
- net LCD_B0: now also U1.D11 (PJ12), J4.17 (Pin_17)
- net LCD_CLK: now also U1.H3 (PI14), J4.28 (Pin_28), TP3.1
- net LCD_DE: now also U1.D7 (PK7), J4.31 (Pin_31), TP6.1
- net LCD_G0: now also U1.N14 (PJ7), J4.9 (Pin_9)
- net LCD_G1: now also U1.N13 (PJ8), J4.10 (Pin_10)
- net LCD_G2: now also U1.M14 (PJ9), J4.11 (Pin_11)
- net LCD_G3: now also U1.L14 (PJ10), J4.12 (Pin_12)
- net LCD_G4: now also U1.K14 (PJ11), J4.13 (Pin_13)
- net LCD_G5: now also U1.A16 (PI0), J4.14 (Pin_14)
- net LCD_G6: now also U1.A15 (PI1), J4.15 (Pin_15)
- net LCD_G7: now also U1.H17 (PK2), J4.16 (Pin_16), TP10.1
- net LCD_HSYNC: now also U1.H1 (PI12), J4.29 (Pin_29), TP4.1
- net LCD_R0: now also U1.P5 (PI15), J4.1 (Pin_1)
- net LCD_R1: now also U1.N6 (PJ0), J4.2 (Pin_2)
- net LCD_R2: now also U1.P6 (PJ1), J4.3 (Pin_3)
- net LCD_R3: now also U1.R13 (PH9), J4.4 (Pin_4)
- net LCD_R4: now also U1.U6 (PJ3), J4.5 (Pin_5)
- net LCD_R5: now also U1.U7 (PJ4), J4.6 (Pin_6)
- net LCD_R6: now also U1.R12 (PJ5), J4.7 (Pin_7)
- net LCD_R7: now also U1.N15 (PJ6), J4.8 (Pin_8), TP9.1
- net LCD_SCL: now also U1.R16 (PD12), J4.33 (Pin_33), TP8.1
- net LCD_SDA: now also U1.R17 (PD13), J4.32 (Pin_32), TP7.1
- net LCD_VSYNC: now also U1.E2 (PI9), J4.30 (Pin_30), TP5.1
- net ROUT0: now also U1.L2 (PC0)
- net ROUT1: now also U1.M2 (PC1)
- net ROUT10: now also U1.A13 (PC10)
- net ROUT11: now also U1.B13 (PC11)
- net ROUT12: now also U1.C12 (PC12)
- net ROUT13: now also U1.E3 (PC13)
- net ROUT14: now also U1.C2 (PC14)
- net ROUT15: now also U1.C1 (PC15)
- net ROUT2: now also U1.M3 (PC2)
- net ROUT3: now also U1.M4 (PC3)
- net ROUT4: now also U1.T4 (PC4)
- net ROUT5: now also U1.U4 (PC5)
- net ROUT6: now also U1.F14 (PC6)
- net ROUT7: now also U1.F13 (PC7)
- net ROUT8: now also U1.E13 (PC8)
- net ROUT9: now also U1.E14 (PC9)
- net at R25.1: now also U1.P16 (PD14); no longer U1.C2 (PC14)
- net LCD_B6: now reaches U1.A8 (PK5)
- net LCD_B6: now also J4.23 (Pin_23)
- net LCD_B3: now reaches U1.B10 (PJ15)
- net LCD_B3: now also J4.20 (Pin_20)
- net LCD_B5: now reaches U1.B8 (PK4)
- net LCD_B5: now also J4.22 (Pin_22)
- net at R26.1: now also U1.P15 (PD15); no longer U1.C1 (PC15)
- net LCD_B7: now reaches U1.C7 (PK6)
- net LCD_B7: now also J4.24 (Pin_24), TP11.1
- net LCD_B4: now reaches U1.C8 (PK3)
- net LCD_B4: now also J4.21 (Pin_21)
- net LCD_B2: now reaches U1.D10 (PJ14)
- net LCD_B2: now also J4.19 (Pin_19)
- net LCD_B1: now reaches U1.E10 (PJ13)
- net LCD_B1: now also J4.18 (Pin_18)
- no-connect marks 17 -> 19
Other:
- note added: "A0"
- note added: "A1"
- note added: "A2"
- note added: "A3"
- note added: "DESERIALIZER CLK wyzwala pojedynczy transfer DMA"
- note added: "I2C"
- note added: "OK"
- note removed: "DODAĆ DO BIBLIOTEKI"
- note removed: "Pododawać testpointy"
- moved on the sheet: C44, C45, C46, C47, C48, C49, C50, C51, C52, C53, C55, J3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

Commit message: Started a bit of routing
Parts:
- added C58: 2.2u, Capacitor_SMD:C_0402_1005Metric, symbol MEMS_CAPACITORS:C_2u2_0402_10V_X5R_LMK105ABJ225KVHF
- added R69, R70: 10k, Resistor_SMD:R_0402_1005Metric, symbol MEMS_RESISTORS_0402:R_10k_0402_1%_50ppm_RT0402FRE0710KL
- added R71, R72: 5k1, Resistor_SMD:R_0402_1005Metric, symbol MEMS_RESISTORS_0402:R_5k1_0402_1%_50ppm_RT0402FRE075K1L
- added R73: 0R, Resistor_SMD:R_0402_1005Metric, symbol MEMS_RESISTORS:R_0R_0402_RMC1/16SJPTH
Connections:
- net GND: now also J3.11 (SHIELD), J3.6 (VSS), J3.9 (DET_B), J6.MP, SW2.1, SW3.1, C58.2
- net VDDA: now also R73.2; no longer C10.1, C11.1, C12.1, C13.1, C14.1, C15.1, C16.1, C17.1, C18.1, C19.1, C20.1, C21.1, C22.1, C23.1, C24.1, C25.1, C26.1, C27.1, C3.1, C4.1, C5.1, C54.1, C6.1, C7.1, C8.1, C9.1, J1.3 (VCC), JP1.2, JP7.2, R64.2, U1.A6 (VDDLDO), U1.B1 (VBAT), U1.C17 (VDDLDO), U1.E11 (VDD), U1.E6 (VDD), U1.E9 (VDD), U1.F17 (VDD33_USB), U1.F5 (VDD), U1.G13 (VDD), U1.G17 (VDD50_USB), U1.G5 (VDD), U1.H13 (VDD), U1.H5 (VDD), U1.J13 (VDD), U1.K13 (VDD), U1.K5 (VDD), U1.L13 (VDD), U1.L5 (VDD), U1.M13 (VDD), U1.M5 (VDD), U1.N10 (VDD), U1.N11 (VDD), U1.N12 (VDD), U1.N7 (VDD), U1.N8 (VDD), U1.P17 (VDD), U1.U12 (VDDLDO)
- net SD_CK: now reaches U1.B11 (PD6)
- net SD_CK: now also J3.5 (CLK)
- net SD_D3: now reaches U1.B7 (PB4)
- net SD_D3: now also J3.2 (DAT3/CD)
- net SD_D2: now reaches U1.B9 (PG11)
- net SD_D2: now also J3.1 (DAT2)
- net SD_CMD: now reaches U1.C11 (PD7)
- net SD_CMD: now also J3.3 (CMD)
- net I2C2_SCL: now reaches U1.P11 (PB10)
- net I2C2_SCL: now also J6.3 (Pin_3), R72.2
- net I2C2_SDA: now reaches U1.P12 (PB11)
- net I2C2_SDA: now also J6.4 (Pin_4), R71.2
- net SD_D1: now reaches U1.T15 (PB15)
- net SD_D1: now also J3.8 (DAT1)
- net SD_D0: now reaches U1.U15 (PB14)
- net SD_D0: now also J3.7 (DAT0)
- net SD_DET_A: now reaches J3.10 (DET_A)
- net VDD_MCU: now reaches J3.4 (VDD)
- net VDD_MCU: now also C10.1, C11.1, C12.1, C13.1, C14.1, C15.1, C16.1, C17.1, C18.1, C19.1, C20.1, C21.1, C22.1, C23.1, C24.1, C25.1, C26.1, C27.1, C3.1, C4.1, C5.1, C54.1, C6.1, C7.1, C8.1, C9.1, J1.3 (VCC), JP1.2, JP7.2, R64.2, U1.A6 (VDDLDO), U1.B1 (VBAT), U1.C17 (VDDLDO), U1.E11 (VDD), U1.E6 (VDD), U1.E9 (VDD), U1.F17 (VDD33_USB), U1.F5 (VDD), U1.G13 (VDD), U1.G17 (VDD50_USB), U1.G5 (VDD), U1.H13 (VDD), U1.H5 (VDD), U1.J13 (VDD), U1.K13 (VDD), U1.K5 (VDD), U1.L13 (VDD), U1.L5 (VDD), U1.M13 (VDD), U1.M5 (VDD), U1.N10 (VDD), U1.N11 (VDD), U1.N12 (VDD), U1.N7 (VDD), U1.N8 (VDD), U1.P17 (VDD), U1.U12 (VDDLDO), C58.1, R71.1, R72.1, R73.1
- net LED_ORANGE: now reaches R63.2
- net at SW2.2: now also R69.1
- net at SW3.2: now also R70.1
- net LED_GREEN: now reaches R62.2
- new net SW_MODE: R70.2
- new net SW_PICTURE: R69.2
Other:
- moved on the sheet: C10, C11, C12, C13, C14, C15, C16, C17, C18, C19, C20, C21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
