File: YTAR/YTAR.kicad_sch (KiCad schematic)
At the start: 167 parts, among them J1 STDC14, J2 CAMERA, J3 Micro_Sd, J4 FH12-40S-0.5SH(55), J5 USB_C_USB4085-GF-A, J6 IO, SW1 RESET, SW2 PICTURE, SW3 MODE, U1 STM32H750XBHx, U2 MCP2562-E-MF, U3 DS90C124, U5 TPS56339, Y1 25MHz

Commit message: Multiple improvements
Parts:
- removed JP2, JP3: ~, MEMS_Passive:R_0805_2012Metric_Jumper_Open, symbol MEMS_PASSIVE:SolderableJumper_Open
- added C59, C64, C67, C68: 100n, Capacitor_SMD:C_0402_1005Metric, symbol MEMS_CAPACITORS:C_100n_0402_16V_X7R_MLASE105SB7104KFNA01
- added C60, C61, C69, C70: 22u, Capacitor_SMD:C_0805_2012Metric, symbol MEMS_CAPACITORS:C_22u_0805_16V_X6S_GRM21BC81C226ME44L
- added C62, C63, C65, C66: 10u, Capacitor_SMD:C_0805_2012Metric, symbol MEMS_CAPACITORS:C_10u_0805_25V_X5R_08053D106KAT4A
- added D5: 3.6V, Diode_SMD:D_SOD-123, symbol MEMS_PROTECTION:D_3V6_ BZT52B3V6-TP
- added D6: 18V, Diode_SMD:D_SOD-123, symbol MEMS_PROTECTION:D_18V_MMSZ4705-HE3_A-08
- added F1: 350mA, Fuse:Fuse_0805_2012Metric, symbol MEMS_PROTECTION:Polyfuse-350mA-0805L035YR
- added F2: Polyfuse-2A-1206L200SLYR, Fuse:Fuse_1206_3216Metric, symbol MEMS_PROTECTION:Polyfuse-2A-1206L200SLYR
- added L1, L2: SRN6028C-6R0M, Inductor_SMD:L_Bourns-SRN6028, symbol MEMS_PASSIVE:SRN6028C-6R0M
- added R74, R75, R78, R82: 33R, Resistor_SMD:R_0402_1005Metric, symbol MEMS_RESISTORS_0402:R_33R_0402_1%_50ppm_RT0402FRE0733RL
- added R76: 52k3, Resistor_SMD:R_0402_1005Metric, symbol MEMS_RESISTORS_0402:R_52k3_0402_1%_50ppm_RT0402FRE0752K3L
- added R77, R81: 10k, Resistor_SMD:R_0402_1005Metric, symbol MEMS_RESISTORS_0402:R_10k_0402_1%_50ppm_RT0402FRE0710KL
- added R79: 0R, Resistor_SMD:R_0402_1005Metric, symbol MEMS_RESISTORS:R_0R_0402_RMC1/16SJPTH
- added R80: 30k9, Resistor_SMD:R_0402_1005Metric, symbol MEMS_RESISTORS_0402:R_30k9_0402_1%_50ppm_RT0402FRE0730K9L
- added TP12: 5V, MEMS_Custom:TestPoint_Pad_D1.0mm, symbol MEMS_ELECTROMECHANICAL:TestPoint
- added TP13: 3V3, MEMS_Custom:TestPoint_Pad_D1.0mm, symbol MEMS_ELECTROMECHANICAL:TestPoint
- added U6: TPS56339, Package_TO_SOT_SMD:TSOT-23-6, symbol MEMS_IC:TPS56339
- JP1: value ~ -> SMPS_5V
- JP4: value ~ -> SMPS_3V3
- TP10: value ~ -> G7
- TP11: value ~ -> B7
- TP3: value ~ -> CLK
- TP4: value ~ -> HSYNC
- TP5: value ~ -> VSYNC
- TP9: value ~ -> R7
Connections:
- net VDD_DES is gone; now on net +3.3V: C46.1, C47.1, C48.1, C49.1, C50.1, C51.1, C52.1, C53.1, R23.2, U3.1 (RPWDNB), U3.20 (VDDOR2), U3.30 (VDDOR1), U3.36 (VDDR0), U3.37 (VDDR1), U3.39 (VDDIR), U3.45 (VDDPR1), U3.47 (VDDPR0), U3.48 (REN), U3.8 (VSSOR3)
- net VDD_DRAM is gone; now on net +3.3V: C29.1, C30.1, C31.1, C32.1, C33.1, C34.1, C35.1, C36.1, C37.1, C38.1, C39.1, C40.1, C41.1, C42.1, U4.A7 (VDD), U4.B2 (VDDQ), U4.B7 (VDDQ), U4.C9 (VDDQ), U4.D9 (VDDQ), U4.E1 (VDDQ), U4.F9 (VDD), U4.L1 (VDDQ), U4.L7 (VDD), U4.M9 (VDDQ), U4.N9 (VDDQ), U4.P2 (VDDQ), U4.P7 (VDDQ), U4.R7 (VDD)
- net +12V_CAM: now also U5.3 (VIN), C62.1, C63.1, C64.1, C65.1, C66.1, C67.1, D6.1 (K), F2.1, U6.3 (VIN)
- net +3.3V: now also C10.1, C11.1, C12.1, C13.1, C14.1, C15.1, C16.1, C17.1, C18.1, C19.1, C20.1, C21.1, C22.1, C23.1, C24.1, C25.1, C26.1, C27.1, C3.1, C4.1, C43.1, C5.1, C54.1, C58.1, C6.1, C7.1, C8.1, C9.1, J1.3 (VCC), J3.4 (VDD), JP7.2, R64.2, R71.1, R72.1, R73.1, U1.A6 (VDDLDO), U1.B1 (VBAT), U1.C17 (VDDLDO), U1.E11 (VDD), U1.E6 (VDD), U1.E9 (VDD), U1.F17 (VDD33_USB), U1.F5 (VDD), U1.G13 (VDD), U1.G17 (VDD50_USB), U1.G5 (VDD), U1.H13 (VDD), U1.H5 (VDD), U1.J13 (VDD), U1.K13 (VDD), U1.K5 (VDD), U1.L13 (VDD), U1.L5 (VDD), U1.M13 (VDD), U1.M5 (VDD), U1.N10 (VDD), U1.N11 (VDD), U1.N12 (VDD), U1.N7 (VDD), U1.N8 (VDD), U1.P17 (VDD), U1.U12 (VDDLDO), U2.3 (VDD), U2.5 (Vio), D5.1 (K), F1.2; no longer JP1.1, JP4.1
- net +5V: now also JP1.1, R79.1; no longer J4.25 (Pin_25), J4.26 (Pin_26)
- net GND: now also J2.MP, J4.MP, U5.1 (GND), C60.2, C61.2, C62.2, C63.2, C64.2, C65.2, C66.2, C67.2, C69.2, C70.2, D5.2 (A), D6.2 (A), R77.2, R81.2, U6.1 (GND)
- net CAM_AUX_A: now reaches J2.7 (Pin_7)
- net CAM_AUX_B: now reaches J2.8 (Pin_8)
- net LCD_PWM: now reaches J4.34 (Pin_34)
- net LCD_AUX_1: now reaches J4.35 (Pin_35)
- net LCD_AUX_2: now reaches J4.36 (Pin_36)
- net LCD_AUX_3: now reaches J4.37 (Pin_37)
- net LCD_AUX_4: now reaches J4.38 (Pin_38)
- net LCD_AUX_5: now reaches J4.39 (Pin_39)
- net at U5.2 (SW): now also L1.1, R74.2
- net at U5.4 (FB): now also R76.2, R77.1
- net at U5.6 (BOOT): now also C59.1
- net IO_AUX_1: now reaches J6.5 (Pin_5)
- net IO_AUX_2: now reaches J6.6 (Pin_6)
- net IO_AUX_3: now reaches J6.7 (Pin_7)
- net IO_AUX_4: now reaches J6.8 (Pin_8)
- net +12V_IN: no longer names the net of J6.1 (Pin_1)
- net +12V_IN: now also F2.2
- removed net VDD_CAN: C43.1, JP4.2, U2.3 (VDD), U2.5 (Vio)
- removed net VDD_MCU: C10.1, C11.1, C12.1, C13.1, C14.1, C15.1, C16.1, C17.1, C18.1, C19.1, C20.1, C21.1, C22.1, C23.1, C24.1, C25.1, C26.1, C27.1, C3.1, C4.1, C5.1, C54.1, C58.1, C6.1, C7.1, C8.1, C9.1, J1.3 (VCC), J3.4 (VDD), JP1.2, JP7.2, R64.2, R71.1, R72.1, R73.1, U1.A6 (VDDLDO), U1.B1 (VBAT), U1.C17 (VDDLDO), U1.E11 (VDD), U1.E6 (VDD), U1.E9 (VDD), U1.F17 (VDD33_USB), U1.F5 (VDD), U1.G13 (VDD), U1.G17 (VDD50_USB), U1.G5 (VDD), U1.H13 (VDD), U1.H5 (VDD), U1.J13 (VDD), U1.K13 (VDD), U1.K5 (VDD), U1.L13 (VDD), U1.L5 (VDD), U1.M13 (VDD), U1.M5 (VDD), U1.N10 (VDD), U1.N11 (VDD), U1.N12 (VDD), U1.N7 (VDD), U1.N8 (VDD), U1.P17 (VDD), U1.U12 (VDDLDO)
- new net: C68.2, R78.1
- new net: L2.1, R78.2, U6.2 (SW)
- new net: R75.1, R80.1
- new net: R80.2, R81.1, U6.4 (FB)
- new net: C60.1, C61.1, JP1.2, L1.2, R82.2, TP12.1
- new net: C68.1, U6.6 (BOOT)
- new net: J4.25 (Pin_25), J4.26 (Pin_26), R79.2
- new net: C69.1, C70.1, JP4.2, L2.2, R75.2, TP13.1
- new net: F1.1, JP4.1
- new net: C59.2, R74.1
- new net: R76.1, R82.1
- no-connect marks 19 -> 24
Other:
- note added: "Co chcemy wyprowadzić mu na mordę?"
- note added: "Do podłączenia po części głównej"
- note added: "SERDES DMA"
- note added: "Sprawdzić czy pinout ma sens i czy coś dodać"
- note removed: "VBAT tymczasowo do 3V3"
- note removed: "ZAMIENIĆ NA COŚ FAJNEGO"
- moved on the sheet: C10, C11, C12, C13, C14, C15, C16, C17, C18, C19, C20, C21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
