File: YTAR/YTAR.kicad_sch (KiCad schematic)
At the start: 195 parts, among them J1 STDC14, J2 CAMERA, J3 Micro_Sd, J4 FH12-40S-0.5SH(55), J5 USB_C_USB4085-GF-A, J6 IO, SW1 RESET, SW2 PICTURE, SW3 MODE, U1 STM32H750XBHx, U2 MCP2562-E-MF, U3 DS90C124, U5 TPS56339, U6 TPS56339, Y1 25MHz

Commit message: Primary layout done
Parts:
- removed D5: 3.6V, Diode_SMD:D_SOD-123, symbol MEMS_PROTECTION:D_3V6_ BZT52B3V6-TP
- removed JP1: SMPS_5V, MEMS_Passive:R_0805_2012Metric_Jumper_Open, symbol MEMS_PASSIVE:SolderableJumper_Open
- removed JP4: SMPS_3V3, MEMS_Passive:R_0805_2012Metric_Jumper_Open, symbol MEMS_PASSIVE:SolderableJumper_Open
- removed JP5: CAN, MEMS_Passive:R_0805_2012Metric_Jumper_Open, symbol MEMS_PASSIVE:SolderableJumper_Open
- removed JP6: DES_CLK_SEL, MEMS_Passive:R_0805_2012Metric_Jumper_Open, symbol MEMS_PASSIVE:SolderableJumper_Open
- removed JP7: BOOT, MEMS_Passive:R_0805_2012Metric_Jumper_Open, symbol MEMS_PASSIVE:SolderableJumper_Open
- removed R73: 0R, Resistor_SMD:R_0402_1005Metric, symbol MEMS_RESISTORS:R_0R_0402_RMC1/16SJPTH
- removed R75, R82: 33R, Resistor_SMD:R_0402_1005Metric, symbol MEMS_RESISTORS_0402:R_33R_0402_1%_50ppm_RT0402FRE0733RL
- removed TP1: Reset, MEMS_Custom:TestPoint_Pad_D1.0mm, symbol MEMS_ELECTROMECHANICAL:TestPoint
- removed TP10: G7, MEMS_Custom:TestPoint_Pad_D1.0mm, symbol MEMS_ELECTROMECHANICAL:TestPoint
- removed TP11: B7, MEMS_Custom:TestPoint_Pad_D1.0mm, symbol MEMS_ELECTROMECHANICAL:TestPoint
- removed TP12: 5V, MEMS_Custom:TestPoint_Pad_D1.0mm, symbol MEMS_ELECTROMECHANICAL:TestPoint
- removed TP13, TP2: 3V3, MEMS_Custom:TestPoint_Pad_D1.0mm, symbol MEMS_ELECTROMECHANICAL:TestPoint
- removed TP3: CLK, MEMS_Custom:TestPoint_Pad_D1.0mm, symbol MEMS_ELECTROMECHANICAL:TestPoint
- removed TP4: HSYNC, MEMS_Custom:TestPoint_Pad_D1.0mm, symbol MEMS_ELECTROMECHANICAL:TestPoint
- removed TP5: VSYNC, MEMS_Custom:TestPoint_Pad_D1.0mm, symbol MEMS_ELECTROMECHANICAL:TestPoint
- removed TP6, TP7, TP8: ~, MEMS_Custom:TestPoint_Pad_D1.0mm, symbol MEMS_ELECTROMECHANICAL:TestPoint
- removed TP9: R7, MEMS_Custom:TestPoint_Pad_D1.0mm, symbol MEMS_ELECTROMECHANICAL:TestPoint
- added D4: 3.6V, Diode_SMD:D_SOD-123, symbol MEMS_PROTECTION:D_3V6_ BZT52B3V6-TP
- added H1, H2: MountingHole_Pad, MountingHole:MountingHole_2.2mm_M2_DIN965_Pad, symbol Mechanical:MountingHole_Pad
- added JP1: 5V, MEMS_Custom:JP_0402_OPEN, symbol MEMS_PASSIVE:SolderableJumper_0402
- added JP2, JP4: RESET, MEMS_Custom:JP_0402_OPEN, symbol MEMS_PASSIVE:SolderableJumper_0402
- added JP3: 3V3, MEMS_Custom:JP_0402_OPEN, symbol MEMS_PASSIVE:SolderableJumper_0402
- added JP5: CAN, MEMS_Custom:JP_0402_OPEN, symbol MEMS_PASSIVE:SolderableJumper_0402
- added JP6: VDDA, MEMS_Custom:JP_0402_OPEN, symbol MEMS_PASSIVE:SolderableJumper_0402
- added R73, R75: 49R9, Resistor_SMD:R_0402_1005Metric, symbol MEMS_RESISTORS_0402:R_49R9_0402_1%_50ppm_RT0402FRE0749R9L
- added R82, R83: 0R, Resistor_SMD:R_0402_1005Metric, symbol MEMS_RESISTORS:R_0R_0402_RMC1/16SJPTH
- added TP1: RESET, MEMS_Custom:TestPoint_Pad_D0.6mm_SMT, symbol MEMS_OTHER:TP_0.6mm_SMT
- added TP10, TP11, TP15, TP16, TP17, TP18, TP19, TP20, TP21, TP22, TP23, TP24, TP25, TP26, TP27, TP28, TP29, TP3, TP30, TP31, TP32, TP33, TP34, TP35, TP36, TP37, TP4, TP5, TP6, TP7, TP8, TP9: ~, MEMS_Custom:TestPoint_Pad_D0.6mm_SMT, symbol MEMS_OTHER:TP_0.6mm_SMT
- added TP12: 5V, MEMS_Custom:TestPoint_Pad_D0.6mm_SMT, symbol MEMS_OTHER:TP_0.6mm_SMT
- added TP13: 3V3, MEMS_Custom:TestPoint_Pad_D0.6mm_SMT, symbol MEMS_OTHER:TP_0.6mm_SMT
- added TP14: VIN, MEMS_Custom:TestPoint_Pad_D0.6mm_SMT, symbol MEMS_OTHER:TP_0.6mm_SMT
- added TP2: 3V3 OUT, MEMS_Custom:TestPoint_Pad_D0.6mm_SMT, symbol MEMS_OTHER:TP_0.6mm_SMT
Connections:
- net +12V_CAM: now also TP14.1
- net +3.3V: now also D4.1 (K), JP2.2, JP6.2, TP13.1
- net +5V: now also JP1.1
- net BOOT0: now also JP2.1
- net CAN_L: now also JP5.1
- net DES_LOCK: now also R83.2; no longer U1.N4 (PA1)
- net DES_RCLK: now also R82.2; no longer U1.N5 (PA0)
- net DES_RRFB: now also JP4.2
- net GND: now also D4.2 (A), H1.1, H2.1, JP4.1
- net IO_AUX_1: now also TP34.1
- net IO_AUX_2: now also TP35.1
- net IO_AUX_3: now also TP36.1
- net IO_AUX_4: now also TP37.1
- net LCD_B7: now also TP5.1
- net LCD_CLK: now also TP6.1
- net LCD_DE: now also TP9.1
- net LCD_G7: now also TP4.1
- net LCD_HSYNC: now also TP7.1
- net LCD_PWM: now also TP15.1
- net LCD_R7: now also TP3.1
- net LCD_SCL: now also TP11.1
- net LCD_SDA: now also TP10.1
- net LCD_VSYNC: now also TP8.1
- net ROUT0: now also TP16.1
- net ROUT1: now also TP17.1
- net ROUT10: now also TP26.1
- net ROUT11: now also TP27.1
- net ROUT12: now also TP28.1
- net ROUT13: now also TP29.1
- net ROUT14: now also TP30.1
- net ROUT15: now also TP31.1
- net ROUT2: now also TP18.1
- net ROUT3: now also TP19.1
- net ROUT4: now also TP20.1
- net ROUT5: now also TP21.1
- net ROUT6: now also TP22.1
- net ROUT7: now also TP23.1
- net ROUT8: now also TP24.1
- net ROUT9: now also TP25.1
- net VDDA: now also JP6.1
- net ~{STM_RST}: now also TP1.1
- net at R80.1: now also R73.2
- net at C60.1, C61.1, L1.2: now also JP1.2, R75.1, TP12.1
- net at C69.1, C70.1, L2.2: now also JP3.2, R73.1, TP2.1
- net at R20.2: now also JP5.2
- net at F1.1: now also JP3.1
- net at R76.1: now also R75.2
- new net: R83.1, TP33.1, U1.N4 (PA1)
- new net: R82.1, TP32.1, U1.N5 (PA0)
Other:
- note added: "3V3 SMPS"
- note added: "5V SMPS"
- note added: "<- Wejście zasilania"
- note added: "CAN DRIVER"
- note added: "DESERIALIZER"
- note added: "JTAG/SWDIO"
- note added: "LCD"
- note added: "MICRO SD"
- note added: "USB"
- moved on the sheet: C10, C11, C12, C13, C14, C15, C16, C17, C18, C19, C20, C21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

Commit message: DRAM routing
Other:
- moved on the sheet: J2
Changed lines of the file:
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@@
 	(wire
 		(pts
-			(xy 41.91 287.02) (xy 27.94 287.02)
+			(xy 41.91 266.7) (xy 27.94 266.7)
 		)
 		(stroke
@@
 	(wire
 		(pts
-			(xy 41.91 289.56) (xy 27.94 289.56)
+			(xy 41.91 269.24) (xy 27.94 269.24)
 		)
 		(stroke
@@
 	(wire
 		(pts
-			(xy 45.72 276.86) (xy 45.72 274.32)
+			(xy 45.72 256.54) (xy 45.72 254)
 		)
 		(stroke
@@
 	(wire
 		(pts
-			(xy 45.72 271.78) (xy 27.94 271.78)
+			(xy 45.72 251.46) (xy 27.94 251.46)
 		)
 		(stroke
@@
 	(wire
 		(pts
-			(xy 45.72 269.24) (xy 45.72 271.78)
+			(xy 45.72 248.92) (xy 45.72 251.46)
 		)
 		(stroke
@@
 	(wire
 		(pts
-			(xy 41.91 279.4) (xy 27.94 279.4)
+			(xy 41.91 259.08) (xy 27.94 259.08)
 		)
 		(stroke
@@
 	(wire
 		(pts
-			(xy 41.91 276.86) (xy 27.94 276.86)
+			(xy 41.91 256.54) (xy 27.94 256.54)
 		)
 		(stroke
@@
 	(wire
 		(pts
-			(xy 41.91 284.48) (xy 27.94 284.48)
+			(xy 41.91 264.16) (xy 27.94 264.16)
 		)
 		(stroke
@@
 	(wire
 		(pts
-			(xy 41.91 281.94) (xy 27.94 281.94)
+			(xy 41.91 261.62) (xy 27.94 261.62)
 		)
 		(stroke
@@
 	(wire
 		(pts
-			(xy 45.72 274.32) (xy 27.94 274.32)
+			(xy 45.72 254) (xy 27.94 254)
 		)
 		(stroke
@@
 	)
 	(label "CAM_LVDS_L"
-		(at 41.91 279.4 180)
+		(at 41.91 259.08 180)
 		(fields_autoplaced yes)
 		(effects
@@
 	)
 	(label "CAM_AUX_B"
-		(at 41.91 289.56 180)
+		(at 41.91 269.24 180)
 		(fields_autoplaced yes)
 		(effects
@@
 	)
 	(label "CAM_LVDS_H"
-		(at 41.91 276.86 180)
+		(at 41.91 256.54 180)
 		(fields_autoplaced yes)
 		(effects
@@
 	)
 	(label "CAM_CAN_L"
-		(at 41.91 284.48 180)
+		(at 41.91 264.16 180)
 		(fields_autoplaced yes)
 		(effects
@@
 	)
 	(label "CAM_AUX_A"
-		(at 41.91 287.02 180)
+		(at 41.91 266.7 180)
 		(fields_autoplaced yes)
 		(effects
@@
 	)
 	(label "CAM_CAN_H"
-		(at 41.91 281.94 180)
+		(at 41.91 261.62 180)
 		(fields_autoplaced yes)
 		(effects
@@
 		(lib_name "DF52-8S-0.8H_1")
 		(lib_id "MEMS_ELECTROMECHANICAL:DF52-8S-0.8H")
-		(at 22.86 279.4 0)
+		(at 22.86 259.08 0)
 		(mirror y)
 		(unit 1)
@@
 		(dnp no)
 		(property "Reference" "J2"
-			(at 20.32 278.1299 0)
+			(at 20.32 257.8099 0)
 			(effects
 				(font
@@
 		)
 		(property "Value" "CAMERA"
-			(at 32.258 292.608 0)
+			(at 32.258 272.288 0)
 			(effects
 				(font
@@
 		)
 		(property "Footprint" "Connector_Hirose:Hirose_DF52-8S-0.8H_1x08-1MP_P0.80mm_Horizontal"
-			(at 22.86 279.4 0)
+			(at 22.86 259.08 0)
 			(effects
 				(font
@@
 		)
 		(property "Datasheet" "https://www.mouser.pl/datasheet/2/185/DF52_10P_0_8C_CL0668_0017_7_00_Catalog_D51171_en-2487017.pdf"
-			(at 22.86 279.4 0)
+			(at 22.86 259.08 0)
 			(effects
 				(font
@@
 		)
 		(property "Description" "To be paired with DF52-8P-0.8C using DF52-2832PCF"
-			(at 22.86 279.4 0)
+			(at 22.86 259.08 0)
 			(effects
 				(font
@@
 		)
 		(property "MPN" " DF52-8S-0.8H(21) "
-			(at 45.466 295.656 0)
+			(at 45.466 275.336 0)
 			(effects
 				(font
@@
 	(symbol
 		(lib_id "power:GND")
-		(at 22.86 293.37 0)
+		(at 22.86 273.05 0)
 		(mirror y)
 		(unit 1)
@@
 		(fields_autoplaced yes)
 		(property "Reference" "#PWR071"
-			(at 22.86 299.72 0)
+			(at 22.86 279.4 0)
 			(effects
 				(font
@@
 		)
 		(property "Value" "GND"
-			(at 22.86 298.45 0)
+			(at 22.86 278.13 0)
 			(effects
 				(font
@@
 		)
 		(property "Footprint" ""
-			(at 22.86 293.37 0)
+			(at 22.86 273.05 0)
 			(effects
 				(font
@@
 		)
 		(property "Datasheet" ""
-			(at 22.86 293.37 0)
+			(at 22.86 273.05 0)
 			(effects
 				(font
@@
 		)
 		(property "Description" "Power symbol creates a global label with name \"GND\" , ground"
-			(at 22.86 293.37 0)
+			(at 22.86 273.05 0)
 			(effects
 				(font
@@
 	(symbol
 		(lib_id "power:GND")
-		(at 45.72 276.86 0)
+		(at 45.72 256.54 0)
 		(mirror y)
 		(unit 1)
@@
 		(fields_autoplaced yes)
 		(property "Reference" "#PWR039"
-			(at 45.72 283.21 0)
+			(at 45.72 262.89 0)
 			(effects
 				(font
@@
 		)
 		(property "Value" "GND"
-			(at 45.72 281.94 0)
+			(at 45.72 261.62 0)
 			(effects
 				(font
@@
 		)
 		(property "Footprint" ""
-			(at 45.72 276.86 0)
+			(at 45.72 256.54 0)
 			(effects
 				(font
@@
 		)
 		(property "Datasheet" ""
-			(at 45.72 276.86 0)
+			(at 45.72 256.54 0)
 			(effects
 				(font
@@
 		)
 		(property "Description" "Power symbol creates a global label with name \"GND\" , ground"
-			(at 45.72 276.86 0)
+			(at 45.72 256.54 0)
 			(effects
 				(font
@@
 	(symbol
 		(lib_id "power:+3.3V")
-		(at 45.72 269.24 0)
+		(at 45.72 248.92 0)
 		(mirror y)
 		(unit 1)
@@
 		(fields_autoplaced yes)
 		(property "Reference" "#PWR_STM011"
-			(at 45.72 273.05 0)
+			(at 45.72 252.73 0)
 			(effects
 				(font
@@
 		)
 		(property "Value" "+12V_CAM"
-			(at 45.72 264.16 0)
+			(at 45.72 243.84 0)
 			(effects
 				(font
@@
 		)
 		(property "Footprint" ""
-			(at 45.72 269.24 0)
+			(at 45.72 248.92 0)
 			(effects
 				(font
@@
 		)
 		(property "Datasheet" ""
-			(at 45.72 269.24 0)
+			(at 45.72 248.92 0)
 			(effects
 				(font
@@
 		)
 		(property "Description" "Power symbol creates a global label with name \"+3.3V\""
-			(at 45.72 269.24 0)
+			(at 45.72 248.92 0)
 			(effects
 				(font

Commit message: Huuuh
Connections:
- net CAN_H is gone; now on net CAM_CAN_H: R20.1, U2.7 (CANH)
- net CAN_L is gone; now on net CAM_CAN_L: JP5.1, U2.6 (CANL)
- net CAN_RX is gone; now on net FD_CAN1_RX: U2.4 (RXD)
- net CAN_TX is gone; now on net FD_CAN1_TX: U2.1 (TXD)
- net FD_CAN1_RX: now also U1.D5 (PB8); no longer U1.B17 (PH14)
- net IO_AUX_1: now also U1.R3 (PA6)
- net IO_AUX_2: now also U1.T3 (PA5)
- no-connect marks 24 -> 88
Other:
- moved on the sheet: JP1

Commit message: Trud skonczon
Parts:
- added C71: 2.2u, Capacitor_SMD:C_0402_1005Metric, symbol MEMS_CAPACITORS:C_2u2_0402_10V_X5R_LMK105ABJ225KVHF
Connections:
- net GND: now also C71.2
- net LCD_AUX_1: now also U1.A5 (PB5)
- net LCD_PWM: now also U1.B5 (PB6)
- net LED_GREEN: now also U1.A4 (PI4)
- net LED_ORANGE: now also U1.A2 (PI6)
- net SD_DET_A: now also U1.R15 (PD11)
- net SW_MODE: now also U1.T14 (PB12)
- net SW_PICTURE: now also U1.U14 (PB13)
- net DCMI_VSYNC: now reaches U1.A3 (PI5)
- net DCMI_D11: now reaches U1.B16 (PH15)
- net DCMI_D4: now reaches U1.B17 (PH14)
- net DCMI_D1: now reaches U1.P13 (PH10)
- net DCMI_D2: now reaches U1.P14 (PH11)
- net DCMI_D3: now reaches U1.R14 (PH12)
- net DCMI_HSYNC: now reaches U1.U3 (PA4)
- net IO_AUX_1 renamed DCMI_PIXCLK
- new net: C1.1, U1.D17 (VCAP)
- new net: C2.1, U1.U11 (VCAP)
- new net: C71.1, U1.A7 (VCAP)
- no-connect marks 88 -> 73

Commit message: Do rewizji
Parts:
- added TP38, TP39, TP40, TP41, TP42, TP43, TP44: ~, MEMS_Custom:TestPoint_Pad_D0.6mm_SMT, symbol MEMS_OTHER:TP_0.6mm_SMT
Connections:
- net LCD_AUX_2 is gone; now on net +3.3V: J4.36 (Pin_36)
- net CAM_AUX_A: now also TP44.1
- net CAM_AUX_B: now also TP43.1
- net DCMI_HSYNC: now also TP41.1
- net LCD_AUX_3: now also TP40.1
- net at U1.H15 (PG3): now also TP39.1
- net at U1.H16 (PG2): now also TP38.1
- net at U1.U2 (PA3): now also TP42.1
- no-connect marks 73 -> 71
Other:
- note removed: "Do podłączenia po części głównej"

Commit message: Dodano TP. Jest ladniej
Parts:
- added TP45, TP46: ~, MEMS_Custom:TestPoint_Pad_D0.6mm_SMT, symbol MEMS_OTHER:TP_0.6mm_SMT
- added TP47: D1, MEMS_Custom:TestPoint_Pad_D0.6mm_SMT, symbol MEMS_OTHER:TP_0.6mm_SMT
- added TP48: D2, MEMS_Custom:TestPoint_Pad_D0.6mm_SMT, symbol MEMS_OTHER:TP_0.6mm_SMT
- added TP49: D3, MEMS_Custom:TestPoint_Pad_D0.6mm_SMT, symbol MEMS_OTHER:TP_0.6mm_SMT
- added TP50: D4, MEMS_Custom:TestPoint_Pad_D0.6mm_SMT, symbol MEMS_OTHER:TP_0.6mm_SMT
- added TP51: D11, MEMS_Custom:TestPoint_Pad_D0.6mm_SMT, symbol MEMS_OTHER:TP_0.6mm_SMT
- added TP52: RX, MEMS_Custom:TestPoint_Pad_D0.6mm_SMT, symbol MEMS_OTHER:TP_0.6mm_SMT
- added TP53: TX, MEMS_Custom:TestPoint_Pad_D0.6mm_SMT, symbol MEMS_OTHER:TP_0.6mm_SMT
- added TP54: GND, MEMS_Custom:TestPoint_Pad_D0.6mm_SMT, symbol MEMS_OTHER:TP_0.6mm_SMT
Connections:
- net DCMI_D1: now also TP47.1
- net DCMI_D11: now also TP51.1
- net DCMI_D2: now also TP48.1
- net DCMI_D3: now also TP49.1
- net DCMI_D4: now also TP50.1
- net DCMI_VSYNC: now also U1.A10 (PG9), TP45.1; no longer U1.A3 (PI5)
- net FD_CAN1_RX: now also TP52.1
- net FD_CAN1_TX: now also TP53.1
- net GND: now also TP54.1
- net LCD_AUX_4: now also TP46.1
Other:
- moved on the sheet: R71, R72

Commit message: Almost ready to fly
Parts:
- removed JP6: VDDA, MEMS_Custom:JP_0402_OPEN, symbol MEMS_PASSIVE:SolderableJumper_0402
- added R84: 0R, Resistor_SMD:R_0402_1005Metric, symbol MEMS_RESISTORS:R_0R_0402_RMC1/16SJPTH
Connections:
- net LCD_AUX_5 is gone; now on net GND: J4.39 (Pin_39)
- net +3.3V: now also R84.1
- net VDDA: now also R84.2
Other:
- moved on the sheet: TP42

Commit message: DEPLOY
Connections:
- net DES_RCLK: now also U1.T13 (PH8)
- no-connect marks 71 -> 70
Changed lines of the file:
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@@
 	)
 	(no_connect
-		(at 109.22 215.9)
-	)
-	(no_connect
 		(at 54.61 375.92)
 	)
@@
 	(wire
 		(pts
+			(xy 97.79 215.9) (xy 109.22 215.9)
+		)
+		(stroke
+			(width 0)
+			(type default)
+		)
+	)
+	(wire
+		(pts
 			(xy 416.56 170.18) (xy 435.61 170.18)
 		)
@@
 		)
 	)
+	(label "DES_RCLK"
+		(at 97.79 215.9 0)
+		(fields_autoplaced yes)
+		(effects
+			(font
+				(size 1.27 1.27)
+			)
+			(justify left bottom)
+		)
+	)
