File: YTAR/YTAR.kicad_pcb (KiCad board)
At the start: 6 copper layers, 50 x 50 mm, 167 parts, among them J1 STDC14, J2 CAMERA, J3 Micro_Sd, J4 FH12-40S-0.5SH(55), J5 USB_C_USB4085-GF-A, J6 IO, SW1 RESET, SW2 PICTURE, SW3 MODE, U1 STM32H750XBHx, U2 MCP2562-E-MF, U3 DS90C124, U5 TPS56339, Y1 25MHz

Commit message: Multiple improvements
Parts:
- removed JP2, JP3: ~, MEMS_Passive:R_0805_2012Metric_Jumper_Open
- added C59: 100n, Capacitor_SMD:C_0402_1005Metric, F.Cu at (55.5, 40.5)
- added C60: 22u, Capacitor_SMD:C_0805_2012Metric, F.Cu at (56.5, 50.5)
- added C61: 22u, Capacitor_SMD:C_0805_2012Metric, F.Cu at (56.5, 48.5)
- added C62: 10u, Capacitor_SMD:C_0805_2012Metric, F.Cu at (49.5, 43.0)
- added C63: 10u, Capacitor_SMD:C_0805_2012Metric, F.Cu at (90.2, 61.4)
- added C64: 100n, Capacitor_SMD:C_0402_1005Metric, F.Cu at (48.0, 43.0)
- added C65: 10u, Capacitor_SMD:C_0805_2012Metric, F.Cu at (51.5, 43.0)
- added C66: 10u, Capacitor_SMD:C_0805_2012Metric, F.Cu at (90.2, 64.4)
- added C67: 100n, Capacitor_SMD:C_0402_1005Metric, F.Cu at (105.7, 53.3)
- added C68: 100n, Capacitor_SMD:C_0402_1005Metric, F.Cu at (105.7, 55.3)
- added C69: 22u, Capacitor_SMD:C_0805_2012Metric, F.Cu at (90.2, 67.4)
- added C70: 22u, Capacitor_SMD:C_0805_2012Metric, F.Cu at (90.2, 70.4)
- added D5: 3.6V, Diode_SMD:D_SOD-123, F.Cu at (27.5, 65.0)
- added D6: 18V, Diode_SMD:D_SOD-123, F.Cu at (27.5, 68.3)
- added F1: 350mA, Fuse:Fuse_0805_2012Metric, F.Cu at (98.1, 63.7)
- added F2: Polyfuse-2A-1206L200SLYR, Fuse:Fuse_1206_3216Metric, F.Cu at (103.1, 68.5)
- added L1: SRN6028C-6R0M, Inductor_SMD:L_Bourns-SRN6028, F.Cu at (51.5, 48.4)
- added L2: SRN6028C-6R0M, Inductor_SMD:L_Bourns-SRN6028, F.Cu at (91.9, 56.1)
- added R74: 33R, Resistor_SMD:R_0402_1005Metric, F.Cu at (53.5, 40.5)
- added R75: 33R, Resistor_SMD:R_0402_1005Metric, F.Cu at (93.9, 60.9)
- added R76: 52k3, Resistor_SMD:R_0402_1005Metric, F.Cu at (56.5, 46.0)
- added R77: 10k, Resistor_SMD:R_0402_1005Metric, F.Cu at (55.5, 46.0)
- added R78: 33R, Resistor_SMD:R_0402_1005Metric, F.Cu at (93.9, 62.9)
- added R79: 0R, Resistor_SMD:R_0402_1005Metric, F.Cu at (26.0, 71.0)
- added R80: 30k9, Resistor_SMD:R_0402_1005Metric, F.Cu at (93.9, 64.8)
- added R81: 10k, Resistor_SMD:R_0402_1005Metric, F.Cu at (93.9, 66.8)
- added R82: 33R, Resistor_SMD:R_0402_1005Metric, F.Cu at (93.9, 68.8)
- added TP12: 5V, MEMS_Custom:TestPoint_Pad_D1.0mm, F.Cu at (70.5, 52.0)
- added TP13: 3V3, MEMS_Custom:TestPoint_Pad_D1.0mm, F.Cu at (97.4, 69.7)
- added U6: TPS56339, Package_TO_SOT_SMD:TSOT-23-6, F.Cu at (102.9, 64.6)
- JP1: value ~ -> SMPS_5V
- JP4: value ~ -> SMPS_3V3
- TP10: value ~ -> G7
- TP11: value ~ -> B7
- TP3: value ~ -> CLK
- TP4: value ~ -> HSYNC
- TP5: value ~ -> VSYNC
- TP9: value ~ -> R7
- moved JP4 99.0 mm to (98.1, 66.7)
- moved JP1 80.8 mm to (81.3, 49.5)
- moved JP6 32.8 mm to (34.6, 45.0)
- moved U5 26.3 mm to (54.5, 43.0)
- moved JP5 15.4 mm to (17.0, 42.5)
- moved C18 6.24 mm to (38.2, 50.9)
- moved C19 6.24 mm to (38.2, 51.8)
- moved C20 6.24 mm to (38.2, 52.7)
- moved C22 6.24 mm to (38.2, 54.6)
- moved C23 6.24 mm to (38.2, 55.5)
- moved C24 6.24 mm to (38.2, 56.5)
- moved C25 6.24 mm to (41.5, 50.6)
- moved C26 6.24 mm to (41.5, 52.6)
- moved C27 6.24 mm to (41.5, 54.5)
- moved C28 6.24 mm to (41.5, 56.5)
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Connections:
- C10 pad 1: VDD_MCU -> +3.3V
- C11 pad 1: VDD_MCU -> +3.3V
- C12 pad 1: VDD_MCU -> +3.3V
- C13 pad 1: VDD_MCU -> +3.3V
- C14 pad 1: VDD_MCU -> +3.3V
- C15 pad 1: VDD_MCU -> +3.3V
- C16 pad 1: VDD_MCU -> +3.3V
- C17 pad 1: VDD_MCU -> +3.3V
- C18 pad 1: VDD_MCU -> +3.3V
- C19 pad 1: VDD_MCU -> +3.3V
- C20 pad 1: VDD_MCU -> +3.3V
- C21 pad 1: VDD_MCU -> +3.3V
- C22 pad 1: VDD_MCU -> +3.3V
- C23 pad 1: VDD_MCU -> +3.3V
- C24 pad 1: VDD_MCU -> +3.3V
- C25 pad 1: VDD_MCU -> +3.3V
- C26 pad 1: VDD_MCU -> +3.3V
- C27 pad 1: VDD_MCU -> +3.3V
- C29 pad 1: VDD_DRAM -> +3.3V
- C3 pad 1: VDD_MCU -> +3.3V
- C30 pad 1: VDD_DRAM -> +3.3V
- C31 pad 1: VDD_DRAM -> +3.3V
- C32 pad 1: VDD_DRAM -> +3.3V
- C33 pad 1: VDD_DRAM -> +3.3V
- C34 pad 1: VDD_DRAM -> +3.3V
- C35 pad 1: VDD_DRAM -> +3.3V
- C36 pad 1: VDD_DRAM -> +3.3V
- C37 pad 1: VDD_DRAM -> +3.3V
- C38 pad 1: VDD_DRAM -> +3.3V
- C39 pad 1: VDD_DRAM -> +3.3V
- C4 pad 1: VDD_MCU -> +3.3V
- C40 pad 1: VDD_DRAM -> +3.3V
- C41 pad 1: VDD_DRAM -> +3.3V
- C42 pad 1: VDD_DRAM -> +3.3V
- C43 pad 1: VDD_CAN -> +3.3V
- C46 pad 1: VDD_DES -> +3.3V
- C47 pad 1: VDD_DES -> +3.3V
- C48 pad 1: VDD_DES -> +3.3V
- C49 pad 1: VDD_DES -> +3.3V
- C5 pad 1: VDD_MCU -> +3.3V
- C50 pad 1: VDD_DES -> +3.3V
- C51 pad 1: VDD_DES -> +3.3V
- C52 pad 1: VDD_DES -> +3.3V
- C53 pad 1: VDD_DES -> +3.3V
- C54 pad 1: VDD_MCU -> +3.3V
- C58 pad 1: VDD_MCU -> +3.3V
- C6 pad 1: VDD_MCU -> +3.3V
- C7 pad 1: VDD_MCU -> +3.3V
- C8 pad 1: VDD_MCU -> +3.3V
- C9 pad 1: VDD_MCU -> +3.3V
- J1 pad 3: VDD_MCU -> +3.3V
- J2 pad 7: unconnected-(J2-Pin_7-Pad7) -> /CAM_AUX_A
- J2 pad 8: unconnected-(J2-Pin_8-Pad8) -> /CAM_AUX_B
- J2 pad MP: unconnected-(J2-PadMP) -> GND
- J3 pad 4: VDD_MCU -> +3.3V
- J4 pad 25: +5V -> Net-(J4-Pin_25)
- J4 pad 26: +5V -> Net-(J4-Pin_25)
- J4 pad 34: unconnected-(J4-Pin_34-Pad34) -> /LCD_PWM
- J4 pad 35: unconnected-(J4-Pin_35-Pad35) -> /LCD_AUX_1
- J4 pad 36: unconnected-(J4-Pin_36-Pad36) -> /LCD_AUX_2
- J4 pad 37: unconnected-(J4-Pin_37-Pad37) -> /LCD_AUX_3
- J4 pad 38: unconnected-(J4-Pin_38-Pad38) -> /LCD_AUX_4
- J4 pad 39: unconnected-(J4-Pin_39-Pad39) -> /LCD_AUX_5
- J4 pad MP: unconnected-(J4-PadMP) -> GND
- J6 pad 1: +12V_IN -> Net-(J6-Pin_1)
- J6 pad 5: unconnected-(J6-Pin_5-Pad5) -> /IO_AUX_1
- J6 pad 6: unconnected-(J6-Pin_6-Pad6) -> /IO_AUX_2
- J6 pad 7: unconnected-(J6-Pin_7-Pad7) -> /IO_AUX_3
- J6 pad 8: unconnected-(J6-Pin_8-Pad8) -> /IO_AUX_4
- JP1 pad 1: +3.3V -> +5V
- JP1 pad 2: VDD_MCU -> Net-(C60-Pad1)
- JP4 pad 1: +3.3V -> Net-(F1-Pad1)
- JP4 pad 2: VDD_CAN -> Net-(C69-Pad1)
- JP7 pad 2: VDD_MCU -> +3.3V
- R23 pad 2: VDD_DES -> +3.3V
- R64 pad 2: VDD_MCU -> +3.3V
- R71 pad 1: VDD_MCU -> +3.3V
- R72 pad 1: VDD_MCU -> +3.3V
- R73 pad 1: VDD_MCU -> +3.3V
- U1 pad A6: VDD_MCU -> +3.3V
- U1 pad B1: VDD_MCU -> +3.3V
- U1 pad C17: VDD_MCU -> +3.3V
- U1 pad E11: VDD_MCU -> +3.3V
- U1 pad E6: VDD_MCU -> +3.3V
- U1 pad E9: VDD_MCU -> +3.3V
- U1 pad F17: VDD_MCU -> +3.3V
- U1 pad F5: VDD_MCU -> +3.3V
- U1 pad G13: VDD_MCU -> +3.3V
- U1 pad G17: VDD_MCU -> +3.3V
- U1 pad G5: VDD_MCU -> +3.3V
- U1 pad H13: VDD_MCU -> +3.3V
- U1 pad H5: VDD_MCU -> +3.3V
- U1 pad J13: VDD_MCU -> +3.3V
- U1 pad K13: VDD_MCU -> +3.3V
- U1 pad K5: VDD_MCU -> +3.3V
- U1 pad L13: VDD_MCU -> +3.3V
- U1 pad L5: VDD_MCU -> +3.3V
- U1 pad M13: VDD_MCU -> +3.3V
- U1 pad M5: VDD_MCU -> +3.3V
- U1 pad N10: VDD_MCU -> +3.3V
- U1 pad N11: VDD_MCU -> +3.3V
- U1 pad N12: VDD_MCU -> +3.3V
- U1 pad N7: VDD_MCU -> +3.3V
- U1 pad N8: VDD_MCU -> +3.3V
- U1 pad P17: VDD_MCU -> +3.3V
- U1 pad U12: VDD_MCU -> +3.3V
- U2 pad 3: VDD_CAN -> +3.3V
- U2 pad 5: VDD_CAN -> +3.3V
- U3 pad 1: VDD_DES -> +3.3V
- U3 pad 20: VDD_DES -> +3.3V
- U3 pad 30: VDD_DES -> +3.3V
- U3 pad 36: VDD_DES -> +3.3V
- U3 pad 37: VDD_DES -> +3.3V
- U3 pad 39: VDD_DES -> +3.3V
- U3 pad 45: VDD_DES -> +3.3V
- U3 pad 47: VDD_DES -> +3.3V
- U3 pad 48: VDD_DES -> +3.3V
- U3 pad 8: VDD_DES -> +3.3V
- U4 pad A7: VDD_DRAM -> +3.3V
- U4 pad B2: VDD_DRAM -> +3.3V
- U4 pad B7: VDD_DRAM -> +3.3V
- U4 pad C9: VDD_DRAM -> +3.3V
- U4 pad D9: VDD_DRAM -> +3.3V
- U4 pad E1: VDD_DRAM -> +3.3V
- U4 pad F9: VDD_DRAM -> +3.3V
- U4 pad L1: VDD_DRAM -> +3.3V
- U4 pad L7: VDD_DRAM -> +3.3V
- U4 pad M9: VDD_DRAM -> +3.3V
- U4 pad N9: VDD_DRAM -> +3.3V
- U4 pad P2: VDD_DRAM -> +3.3V
- U4 pad P7: VDD_DRAM -> +3.3V
- U4 pad R7: VDD_DRAM -> +3.3V
- U5 pad 1: unconnected-(U5-GND-Pad1) -> GND
- U5 pad 2: unconnected-(U5-SW-Pad2) -> Net-(U5-SW)
- U5 pad 3: unconnected-(U5-VIN-Pad3) -> +12V_CAM
- U5 pad 4: unconnected-(U5-FB-Pad4) -> Net-(U5-FB)
- U5 pad 6: unconnected-(U5-BOOT-Pad6) -> Net-(U5-BOOT)
Routing:
- net VDD_MCU: vias 27 -> 0
- net VDD_DRAM: vias 14 -> 0
- net +3.3V: vias 0 -> 41
- added copper zone on In4.Cu, net +3.3V
- removed copper zone on In4.Cu, net VDD_MCU

Commit message: Primary layout done
Parts:
- removed D5: 3.6V, Diode_SMD:D_SOD-123
- removed JP7: BOOT, MEMS_Passive:R_0805_2012Metric_Jumper_Open
- added D4: 3.6V, Diode_SMD:D_SOD-123, B.Cu at (21.0, 45.1)
- added H1: MountingHole_Pad, MountingHole:MountingHole_2.2mm_M2_DIN965_Pad, F.Cu at (15.5, 58.6)
- added H2: MountingHole_Pad, MountingHole:MountingHole_2.2mm_M2_DIN965_Pad, F.Cu at (59.0, 40.0)
- added JP2: RESET, MEMS_Custom:JP_0402_OPEN, F.Cu at (25.5, 19.5)
- added JP3: 3V3, MEMS_Custom:JP_0402_OPEN, F.Cu at (37.5, 57.0)
- added R83: 0R, Resistor_SMD:R_0402_1005Metric, F.Cu at (25.0, 42.0)
- added TP14: VIN, MEMS_Custom:TestPoint_Pad_D0.6mm_SMT, F.Cu at (31.5, 75.0)
- added TP15: ~, MEMS_Custom:TestPoint_Pad_D0.6mm_SMT, F.Cu at (31.5, 77.2)
- added TP16: ~, MEMS_Custom:TestPoint_Pad_D0.6mm_SMT, F.Cu at (31.5, 79.5)
- added TP17: ~, MEMS_Custom:TestPoint_Pad_D0.6mm_SMT, F.Cu at (31.5, 81.8)
- added TP18: ~, MEMS_Custom:TestPoint_Pad_D0.6mm_SMT, F.Cu at (33.8, 73.0)
- added TP19: ~, MEMS_Custom:TestPoint_Pad_D0.6mm_SMT, F.Cu at (33.8, 75.0)
- added TP20: ~, MEMS_Custom:TestPoint_Pad_D0.6mm_SMT, F.Cu at (33.8, 77.2)
- added TP21: ~, MEMS_Custom:TestPoint_Pad_D0.6mm_SMT, F.Cu at (33.8, 79.5)
- added TP22: ~, MEMS_Custom:TestPoint_Pad_D0.6mm_SMT, F.Cu at (33.8, 81.8)
- added TP23: ~, MEMS_Custom:TestPoint_Pad_D0.6mm_SMT, F.Cu at (36.0, 72.8)
- added TP24: ~, MEMS_Custom:TestPoint_Pad_D0.6mm_SMT, F.Cu at (36.0, 75.0)
- added TP25: ~, MEMS_Custom:TestPoint_Pad_D0.6mm_SMT, F.Cu at (36.0, 77.2)
- added TP26: ~, MEMS_Custom:TestPoint_Pad_D0.6mm_SMT, F.Cu at (36.0, 79.5)
- added TP27: ~, MEMS_Custom:TestPoint_Pad_D0.6mm_SMT, F.Cu at (36.0, 81.8)
- added TP28: ~, MEMS_Custom:TestPoint_Pad_D0.6mm_SMT, F.Cu at (38.2, 72.8)
- added TP29: ~, MEMS_Custom:TestPoint_Pad_D0.6mm_SMT, F.Cu at (38.2, 75.0)
- added TP30: ~, MEMS_Custom:TestPoint_Pad_D0.6mm_SMT, F.Cu at (38.2, 77.2)
- added TP31: ~, MEMS_Custom:TestPoint_Pad_D0.6mm_SMT, F.Cu at (38.2, 79.5)
- added TP32: ~, MEMS_Custom:TestPoint_Pad_D0.6mm_SMT, F.Cu at (38.2, 81.8)
- added TP33: ~, MEMS_Custom:TestPoint_Pad_D0.6mm_SMT, F.Cu at (40.5, 72.8)
- added TP34: ~, MEMS_Custom:TestPoint_Pad_D0.6mm_SMT, F.Cu at (40.5, 75.0)
- added TP35: ~, MEMS_Custom:TestPoint_Pad_D0.6mm_SMT, F.Cu at (40.5, 77.2)
- added TP36: ~, MEMS_Custom:TestPoint_Pad_D0.6mm_SMT, F.Cu at (40.5, 79.5)
- added TP37: ~, MEMS_Custom:TestPoint_Pad_D0.6mm_SMT, F.Cu at (40.5, 81.8)
- C1, C11, C2, C21, C22, C23, C24, C46, C47, C48, C49, C50, C51, C52, C53, C54, C58, D6, F2: moved to B.Cu
- JP1: value SMPS_5V -> 5V; footprint MEMS_Passive:R_0805_2012Metric_Jumper_Open -> MEMS_Custom:JP_0402_OPEN
- JP4: value SMPS_3V3 -> RESET; footprint MEMS_Passive:R_0805_2012Metric_Jumper_Open -> MEMS_Custom:JP_0402_OPEN
- JP5: footprint MEMS_Passive:R_0805_2012Metric_Jumper_Open -> MEMS_Custom:JP_0402_OPEN
- JP6: value DES_CLK_SEL -> VDDA; footprint MEMS_Passive:R_0805_2012Metric_Jumper_Open -> MEMS_Custom:JP_0402_OPEN
- R73: value 0R -> 49R9
- R75: value 33R -> 49R9
- R82: value 33R -> 0R
- TP1: value Reset -> RESET; footprint MEMS_Custom:TestPoint_Pad_D1.0mm -> MEMS_Custom:TestPoint_Pad_D0.6mm_SMT
- TP10: value G7 -> ~; footprint MEMS_Custom:TestPoint_Pad_D1.0mm -> MEMS_Custom:TestPoint_Pad_D0.6mm_SMT
- TP11: value B7 -> ~; footprint MEMS_Custom:TestPoint_Pad_D1.0mm -> MEMS_Custom:TestPoint_Pad_D0.6mm_SMT
- TP12, TP13, TP6, TP7, TP8: footprint MEMS_Custom:TestPoint_Pad_D1.0mm -> MEMS_Custom:TestPoint_Pad_D0.6mm_SMT
- TP2: value 3V3 -> 3V3 OUT; footprint MEMS_Custom:TestPoint_Pad_D1.0mm -> MEMS_Custom:TestPoint_Pad_D0.6mm_SMT
- TP3: value CLK -> ~; footprint MEMS_Custom:TestPoint_Pad_D1.0mm -> MEMS_Custom:TestPoint_Pad_D0.6mm_SMT
- TP4: value HSYNC -> ~; footprint MEMS_Custom:TestPoint_Pad_D1.0mm -> MEMS_Custom:TestPoint_Pad_D0.6mm_SMT
- TP5: value VSYNC -> ~; footprint MEMS_Custom:TestPoint_Pad_D1.0mm -> MEMS_Custom:TestPoint_Pad_D0.6mm_SMT
- TP9: value R7 -> ~; footprint MEMS_Custom:TestPoint_Pad_D1.0mm -> MEMS_Custom:TestPoint_Pad_D0.6mm_SMT
- moved F2 87.8 mm to (18.5, 45.1), turned to 90 degrees
- moved TP13 79.4 mm to (19.5, 54.5)
- moved JP4 76.8 mm to (25.0, 43.0)
- moved R82 74.3 mm to (25.0, 41.0)
- moved TP9 71.8 mm to (29.2, 79.5)
- moved TP10 71.0 mm to (29.2, 81.8)
- moved TP3 70.9 mm to (27.0, 77.2)
- moved TP4 70.2 mm to (27.0, 79.5)
- moved TP5 69.4 mm to (27.0, 81.8)
- moved C68 66.8 mm to (39.5, 46.5), turned to 180 degrees
- moved TP6 66.4 mm to (29.2, 72.8)
- moved TP7 65.7 mm to (29.2, 75.0)
- moved TP8 64.9 mm to (29.2, 77.2)
- moved U6 63.2 mm to (41.5, 49.5), turned to 90 degrees
- moved F1 61.9 mm to (37.0, 53.4), turned to 90 degrees
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Connections:
- JP4 pad 1: Net-(F1-Pad1) -> GND
- JP4 pad 2: Net-(C69-Pad1) -> /DES_RRFB
- JP6 pad 1: GND -> VDDA
- JP6 pad 2: /DES_RRFB -> +3.3V
- R73 pad 1: +3.3V -> Net-(C69-Pad1)
- R73 pad 2: VDDA -> Net-(R73-Pad2)
- R75 pad 1: Net-(R75-Pad1) -> Net-(C60-Pad1)
- R75 pad 2: Net-(C69-Pad1) -> Net-(R75-Pad2)
- R76 pad 1: Net-(R76-Pad1) -> Net-(R75-Pad2)
- R80 pad 1: Net-(R75-Pad1) -> Net-(R73-Pad2)
- R82 pad 1: Net-(R76-Pad1) -> Net-(U1-PA0)
- R82 pad 2: Net-(C60-Pad1) -> /DES_RCLK
- TP10 pad 1: /LCD_G7 -> /LCD_SDA
- TP11 pad 1: /LCD_B7 -> /LCD_SCL
- TP13 pad 1: Net-(C69-Pad1) -> +3.3V
- TP2 pad 1: +3.3V -> Net-(C69-Pad1)
- TP3 pad 1: /LCD_CLK -> /LCD_R7
- TP4 pad 1: /LCD_HSYNC -> /LCD_G7
- TP5 pad 1: /LCD_VSYNC -> /LCD_B7
- TP6 pad 1: /LCD_DE -> /LCD_CLK
- TP7 pad 1: /LCD_SDA -> /LCD_HSYNC
- TP8 pad 1: /LCD_SCL -> /LCD_VSYNC
- TP9 pad 1: /LCD_R7 -> /LCD_DE
- U1 pad N4: /DES_LOCK -> Net-(U1-PA1)
- U1 pad N5: /DES_RCLK -> Net-(U1-PA0)
Routing:
- net Net-(U1-PA1): vias 0 -> 1
- net Net-(U1-PA0): vias 0 -> 1
- net /DES_RCLK: vias 1 -> 0
- net /DES_LOCK: vias 1 -> 0
- added copper zone on In1.Cu, net GND
- added copper zone on In3.Cu, net GND

Commit message: DRAM routing
Parts:
- moved R2 11.4 mm to (55.5, 22.5), turned to 90 degrees
- moved C42 7.61 mm to (58.5, 35.5), turned to 0 degrees
- moved C32 7.34 mm to (47.0, 33.6)
- moved C39 5.84 mm to (52.1, 36.7)
- moved C33 5.75 mm to (58.5, 29.5), turned to 0 degrees
- moved R4 5.50 mm to (46.5, 22.5)
- moved C31 4.85 mm to (58.5, 27.5), turned to 0 degrees
- moved C34 4.77 mm to (58.5, 33.7), turned to 0 degrees
- moved C38 4.72 mm to (47.0, 26.5)
- moved C35 4.61 mm to (52.1, 33.6)
- moved C40 4.39 mm to (47.0, 34.8)
- moved C37 4.35 mm to (47.0, 28.7)
- moved R6 3.50 mm to (47.5, 22.5)
- moved R1 2.00 mm to (50.5, 22.5), turned to 90 degrees
- moved R79 1.74 mm to (44.5, 21.6)
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Routing:
- net /SDN_CAS: track 0.00 -> 34.1 mm, vias 0 -> 4
- net /DQ2: track 0.00 -> 32.5 mm, vias 0 -> 3
- net /DQ3: track 0.00 -> 28.0 mm, vias 0 -> 3
- net +3.3V: track 0.00 -> 27.6 mm, vias 41 -> 42
- net /DQ7: track 0.00 -> 22.6 mm, vias 0 -> 4
- net /BA1: track 0.00 -> 22.3 mm, vias 0 -> 4
- net /DQ6: track 0.00 -> 19.3 mm, vias 0 -> 3
- net /DQ4: track 0.00 -> 18.9 mm, vias 0 -> 2
- net /BA0: track 0.00 -> 18.7 mm, vias 0 -> 4
- net /DQ5: track 0.00 -> 18.0 mm, vias 0 -> 4
- net /SDN_CLK: track 0.00 -> 17.9 mm, vias 0 -> 4
- net /SDN_NE: track 0.00 -> 17.3 mm, vias 0 -> 3
- net /A0: track 0.00 -> 16.3 mm, vias 0 -> 3
- net /DQ9: track 0.00 -> 16.1 mm, vias 0 -> 3
- net /A1: track 0.00 -> 15.7 mm, vias 0 -> 3
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- added copper zone on B.Cu, net GND
